File: z80_computer.sch (KiCad schematic (older format))
At the start: 61 parts, among them J1 Barrel_Jack_MountingPin, J12 +5V, SW1 RESET, SW2 Power Switch, SW6 Soft Pwr, U1 74HCT04, U2 NE555P, U3 LM2576HVS-ADJ, U4 74LS74, U5 AMS1117-3.3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

Commit message: Fixed up issues
Parts:
- added H7: Placeholder Graphic, Symbol:Symbol_Barrel_Polarity, symbol Mechanical:MountingHole
- D2: value Green -> Power
- J1: value Barrel_Jack_MountingPin -> 7-25v
- SW2: value Power Switch -> Power OFF - ON
- SW6: value Soft Pwr -> Soft Power
- TP6: value 3v3 -> 3.3v
Changed lines of the file:
@@
 U 2 1 60178610
 P 2250 3700
-F 0 "U1" H 2250 4017 50  0000 C CNN
+F 0 "U1" V 2250 4017 50  0000 C CNN
 F 1 "74HCT04" H 2250 3926 50  0000 C CNN
 F 2 "Package_DIP:DIP-14_W7.62mm_Socket" H 2250 3700 50  0001 C CNN
@@
 P 5500 2000
 F 0 "D2" V 5539 1882 50  0000 R CNN
-F 1 "Green" V 5448 1882 50  0000 R CNN
+F 1 "Power" V 5448 1882 50  0000 R CNN
 F 2 "LED_THT:LED_D5.0mm" H 5500 2000 50  0001 C CNN
 F 3 "~" H 5500 2000 50  0001 C CNN
@@
 P 1650 1300
 F 0 "SW2" H 1650 1585 50  0000 C CNN
-F 1 "Power Switch" H 1650 1494 50  0000 C CNN
+F 1 "Power OFF - ON" H 1650 1494 50  0000 C CNN
 F 2 "Button_Switch_THT:SW_Slide_1P2T_CK_OS102011MS2Q" H 1650 1300 50  0001 C CNN
 F 3 "~" H 1650 1300 50  0001 C CNN
@@
 P 8550 1350
 F 0 "TP6" H 8608 1468 50  0000 L CNN
-F 1 "3v3" H 8608 1377 50  0000 L CNN
+F 1 "3.3v" H 8608 1377 50  0000 L CNN
 F 2 "TestPoint:TestPoint_Pad_D2.0mm" H 8750 1350 50  0001 C CNN
 F 3 "~" H 8750 1350 50  0001 C CNN
@@
 P 1050 1300
 F 0 "J1" H 1107 1617 50  0000 C CNN
-F 1 "Barrel_Jack_MountingPin" H 1107 1526 50  0000 C CNN
+F 1 "7-25v" H 1107 1526 50  0000 C CNN
 F 2 "Connector_BarrelJack:BarrelJack_Horizontal" H 1100 1260 50  0001 C CNN
 F 3 "~" H 1100 1260 50  0001 C CNN
@@
 P 2550 1900
 F 0 "SW6" H 2550 2185 50  0000 C CNN
-F 1 "Soft Pwr" H 2550 1700 50  0000 C CNN
+F 1 "Soft Power" H 2550 1700 50  0000 C CNN
 F 2 "Button_Switch_THT:SW_Slide_1P2T_CK_OS102011MS2Q" H 2550 1900 50  0001 C CNN
 F 3 "~" H 2550 1900 50  0001 C CNN
@@
 Wire Wire Line
 	7950 4400 8350 4400
+$Comp
+L Mechanical:MountingHole H7
+U 1 1 6127328F
+P 850 1750
+F 0 "H7" H 950 1796 50  0000 L CNN
+F 1 "Placeholder Graphic" H 950 1705 50  0000 L CNN
+F 2 "Symbol:Symbol_Barrel_Polarity" H 850 1750 50  0001 C CNN
+F 3 "~" H 850 1750 50  0001 C CNN
+	1    850  1750
+	1    0    0    -1
+$EndComp
 $EndSCHEMATC
