File: z80_computer.sch (KiCad schematic (older format))
At the start: 62 parts, among them J1 7-25v, J12 +5V, SW1 RESET, SW2 Power OFF - ON, SW6 Soft Power, U1 74HCT04, U2 NE555P, U3 LM2576HVS-ADJ, U4 74LS74, U5 AMS1117-3.3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

Commit message: Bug fixes. Moved components two new sheet; added voltage monitor for RTC
Parts:
- removed SW6: Soft Power, Button_Switch_THT:SW_Slide_1P2T_CK_OS102011MS2Q, symbol Switch:SW_SPDT
Connections:
- net +5V: no longer TP5.1
- net GND: now also U3.5 (~ON~/OFF)
- net at C7.1, JP1.1, L1.2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: now also TP5.1
Other:
- moved on the sheet: H7, TP5
Changed lines of the file:
@@
 $Descr A4 11693 8268
 encoding utf-8
-Sheet 1 5
+Sheet 1 6
 Title "Z80 Computer"
 Date "2021-02-02"
@@
 Connection ~ 3750 2200
 $Comp
-L Device:R R7
-U 1 1 6027A198
-P 5050 1650
-F 0 "R7" H 5120 1696 50  0000 L CNN
-F 1 "11k" H 5120 1605 50  0000 L CNN
-F 2 "Resistor_THT:R_Axial_DIN0207_L6.3mm_D2.5mm_P10.16mm_Horizontal" V 4980 1650 50  0001 C CNN
-F 3 "~" H 5050 1650 50  0001 C CNN
-	1    5050 1650
-	1    0    0    -1
-$EndComp
-$Comp
 L Device:R R8
 U 1 1 6027A741
@@
 $EndComp
 Wire Wire Line
-	5050 1800 5050 1850
-Wire Wire Line
-	5050 1850 4900 1850
-Wire Wire Line
 	4900 1850 4900 1300
 Wire Wire Line
 	4900 1300 3500 1300
-Connection ~ 5050 1850
 Wire Wire Line
 	5050 1850 5050 1900
-Wire Wire Line
-	5050 1500 4500 1500
 Connection ~ 4500 1500
 Wire Wire Line
@@
 	0    -1   -1   0
 $EndComp
-Wire Wire Line
-	5050 1500 5200 1500
 Connection ~ 5500 1500
 $Comp
@@
 	1    0    0    -1
 $EndComp
-Text GLabel 3200 2100 2    50   Input ~ 0
-~PWR
 Wire Notes Line
 	6800 750  9350 750
@@
 	5400 1500 5500 1500
 Wire Wire Line
-	5500 1500 5700 1500
-Wire Wire Line
 	6000 1500 6000 1700
 Wire Wire Line
@@
 L Connector:TestPoint TP5
 U 1 1 60658538
-P 5700 1500
-F 0 "TP5" H 5758 1618 50  0000 L CNN
-F 1 "5v" H 5758 1527 50  0000 L CNN
-F 2 "TestPoint:TestPoint_Pad_D2.0mm" H 5900 1500 50  0001 C CNN
-F 3 "~" H 5900 1500 50  0001 C CNN
-	1    5700 1500
-	1    0    0    -1
-$EndComp
-Connection ~ 5700 1500
-Wire Wire Line
-	5700 1500 6000 1500
+P 5050 1150
+F 0 "TP5" H 5108 1268 50  0000 L CNN
+F 1 "5v" H 5108 1177 50  0000 L CNN
+F 2 "TestPoint:TestPoint_Pad_D2.0mm" H 5250 1150 50  0001 C CNN
+F 3 "~" H 5250 1150 50  0001 C CNN
+	1    5050 1150
+	1    0    0    -1
+$EndComp
 $Comp
 L Connector:TestPoint TP1
@@
 $EndComp
 Connection ~ 1350 1400
-$Comp
-L Switch:SW_SPDT SW6
-U 1 1 608BB29F
-P 2550 1900
-F 0 "SW6" H 2550 2185 50  0000 C CNN
-F 1 "Soft Power" H 2550 1700 50  0000 C CNN
-F 2 "Button_Switch_THT:SW_Slide_1P2T_CK_OS102011MS2Q" H 2550 1900 50  0001 C CNN
-F 3 "~" H 2550 1900 50  0001 C CNN
-	1    2550 1900
-	0    -1   1    0
-$EndComp
-Wire Wire Line
-	2450 1500 2450 1700
-Wire Wire Line
-	2450 1700 2550 1700
-Wire Wire Line
-	2650 2100 3200 2100
-Wire Wire Line
-	2450 2100 2450 2200
 Connection ~ 2450 2200
 Wire Wire Line
@@
 L Mechanical:MountingHole H7
 U 1 1 6127328F
-P 850 1750
-F 0 "H7" H 950 1796 50  0000 L CNN
-F 1 "Placeholder Graphic" H 950 1705 50  0000 L CNN
-F 2 "Symbol:Symbol_Barrel_Polarity" H 850 1750 50  0001 C CNN
-F 3 "~" H 850 1750 50  0001 C CNN
-	1    850  1750
+P 10100 2250
+F 0 "H7" H 10200 2296 50  0000 L CNN
+F 1 "Placeholder Graphic" H 10200 2205 50  0000 L CNN
+F 2 "Symbol:Symbol_Barrel_Polarity" H 10100 2250 50  0001 C CNN
+F 3 "~" H 10100 2250 50  0001 C CNN
+	1    10100 2250
 	1    0    0    -1
 $EndComp
@@
 	1    0    0    -1
 $EndComp
+Wire Wire Line
+	2450 1500 2450 2200
+Wire Wire Line
+	5500 1500 6000 1500
+Wire Wire Line
+	5050 1150 5050 1500
+Wire Wire Line
+	5050 1500 4500 1500
+Wire Wire Line
+	5050 1500 5200 1500
+Wire Wire Line
+	5050 1850 4900 1850
+Connection ~ 5050 1850
+Wire Wire Line
+	5050 1800 5050 1850
+$Comp
+L Device:R R7
+U 1 1 6027A198
+P 5050 1650
+F 0 "R7" H 5120 1696 50  0000 L CNN
+F 1 "11k" H 5120 1605 50  0000 L CNN
+F 2 "Resistor_THT:R_Axial_DIN0207_L6.3mm_D2.5mm_P10.16mm_Horizontal" V 4980 1650 50  0001 C CNN
+F 3 "~" H 5050 1650 50  0001 C CNN
+	1    5050 1650
+	1    0    0    -1
+$EndComp
+$Sheet
+S 11950 4900 2200 500
+U 6104856E
+F0 "RTC & Compact Flash" 50
+F1 "RTC_CompactFlash.sch" 50
+$EndSheet
 $EndSCHEMATC
