File: soundlcd.sch (KiCad schematic (older format))
At the start: 36 parts, among them J10 Speaker, J8 GPIO3, J9 Audio out, SW3 BTN 1, SW4 BTN 2, U1 74HCT04, U13 AY-3-8910, U19 RTC72421, U20 ULN2803A, U21 74HC245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

Commit message: buf fixes
Parts:
- added R?: 10k, Resistor_THT:R_Axial_DIN0207_L6.3mm_D2.5mm_P10.16mm_Horizontal, symbol Device:R
Connections:
- net +5V: now also R?.1
- net at U1.9, U20.18 (O1): now also R?.2
Changed lines of the file:
@@
 	4550 1700 4550 1950
 Wire Wire Line
-	4550 1700 4800 1700
+	4550 1700 4650 1700
 Wire Wire Line
 	4800 1700 4800 1950
@@
 Connection ~ 5700 1250
 Wire Wire Line
-	4200 3000 4900 3000
+	4200 3000 4650 3000
 Wire Notes Line
 	750  650  5250 650
@@
 Wire Wire Line
 	10150 3900 10350 3900
+$Comp
+L Device:R R?
+U 1 1 6077F3CF
+P 4650 2850
+F 0 "R?" H 4720 2896 50  0000 L CNN
+F 1 "10k" H 4720 2805 50  0000 L CNN
+F 2 "Resistor_THT:R_Axial_DIN0207_L6.3mm_D2.5mm_P10.16mm_Horizontal" V 4580 2850 50  0001 C CNN
+F 3 "~" H 4650 2850 50  0001 C CNN
+	1    4650 2850
+	1    0    0    -1
+$EndComp
+Connection ~ 4650 3000
+Wire Wire Line
+	4650 3000 4900 3000
+Wire Wire Line
+	4650 2700 4650 1700
 Wire Bus Line
 	2250 6000 2250 6400
@@
 Wire Bus Line
 	1550 2850 1550 3600
+Connection ~ 4650 1700
+Wire Wire Line
+	4650 1700 4800 1700
 $EndSCHEMATC
