File: cpu.sch (KiCad schematic (older format))
At the start: 8 parts, among them SW5 NMI, U15 Z80CPU, U16 GAL16V8, U17 GAL16V8

Commit message: Bug fixes. Moved components two new sheet; added voltage monitor for RTC
Connections:
- net ~INT: now also R15.2, U15.16 (~INT~); no longer R16.2, U15.17 (~NMI~)
- net ~NMI: now also R16.2, U15.17 (~NMI~); no longer R15.2, U15.16 (~INT~)
Changed lines of the file:
@@
 $Descr A4 11693 8268
 encoding utf-8
-Sheet 5 5
+Sheet 5 6
 Title "Z80 CPU & Memory Logic"
 Date "2021-02-02"
@@
 Wire Wire Line
 	1900 2500 1550 2500
-Text GLabel 1550 2500 0    50   Input ~ 0
+Text GLabel 1350 2350 0    50   Input ~ 0
 ~INT
 Wire Wire Line
@@
 Wire Wire Line
 	1350 2350 1600 2350
-Text GLabel 1350 2350 0    50   Input ~ 0
+Text GLabel 1550 2500 0    50   Input ~ 0
 ~NMI
 Text GLabel 1350 3150 0    50   Input ~ 0
